Commit message: Add S5 Max ROS model and integrated demo tools

File: urdf/materials.xacro (robot description, xacro)
@@ -1,6 +1,6 @@
 <?xml version="1.0"?>
 <robot xmlns:xacro="http://www.ros.org/wiki/xacro">
-  <material name="s5max_black">
-    <color rgba="0.03 0.03 0.03 1.0"/>
+  <material name="s5max_body">
+    <color rgba="0.62 0.62 0.64 1.0"/>
   </material>
   <material name="s5max_dark_grey">
@@ -10,3 +10,6 @@
     <color rgba="0.35 0.05 0.05 1.0"/>
   </material>
+  <material name="s5max_front">
+    <color rgba="0.95 0.45 0.05 1.0"/>
+  </material>
 </robot>

File: urdf/robot.urdf.xacro (robot description, xacro)
@@ -17,5 +17,13 @@
         <cylinder radius="${body_radius}" length="${body_height}"/>
       </geometry>
-      <material name="s5max_black"/>
+      <material name="s5max_body"/>
+    </visual>
+    <!-- Temporary orientation marker. The orange mark points forward (+X). -->
+    <visual>
+      <origin xyz="${body_radius * 0.72} 0 ${body_height + 0.001}" rpy="0 0 0"/>
+      <geometry>
+        <box size="0.050 0.012 0.002"/>
+      </geometry>
+      <material name="s5max_front"/>
     </visual>
     <collision>
