Commit message: Add physical S5 Max RViz monitoring

File: urdf/params.xacro (robot description, xacro)
@@ -17,5 +17,5 @@
   <xacro:property name="caster_x" value="0.125"/>
   <xacro:property name="caster_diameter" value="0.025"/>
-  <xacro:property name="lidar_x" value="-0.060"/>
+  <xacro:property name="lidar_x" value="0.060"/>
   <xacro:property name="lidar_y" value="0.000"/>
   <xacro:property name="lidar_diameter" value="0.075"/>

Commit message: fix(docking): align S5 Max hardware docking

File: urdf/params.xacro (robot description, xacro)
@@ -21,4 +21,12 @@
   <xacro:property name="lidar_diameter" value="0.075"/>
   <xacro:property name="lidar_height" value="0.0165"/>
+  <!-- Dock IR receiver poses. Replace these photograph-based positions with
+       direct measurements during physical calibration. -->
+  <xacro:property name="dock_ir_front_x" value="0.174"/>
+  <xacro:property name="dock_ir_front_y" value="0.000"/>
+  <xacro:property name="dock_ir_front_yaw" value="0.000"/>
+  <xacro:property name="dock_ir_right_x" value="0.124"/>
+  <xacro:property name="dock_ir_right_y" value="-0.124"/>
+  <xacro:property name="dock_ir_right_yaw" value="${-pi / 4}"/>
   <!-- Approximate component masses sum to the published total mass. -->
   <xacro:property name="body_mass" value="3.15"/>

File: urdf/robot.urdf.xacro (robot description, xacro)
@@ -113,3 +113,29 @@
     <xacro:solid_cylinder_inertia mass="${lidar_mass}" radius="${lidar_diameter / 2}" length="${lidar_height}"/>
   </link>
+  <joint name="dock_ir_front_joint" type="fixed">
+    <parent link="base_link"/>
+    <child link="dock_ir_front_link"/>
+    <origin xyz="${dock_ir_front_x} ${dock_ir_front_y} ${body_height / 2}" rpy="0 0 ${dock_ir_front_yaw}"/>
+  </joint>
+  <link name="dock_ir_front_link">
+    <visual>
+      <geometry>
+        <box size="0.006 0.020 0.012"/>
+      </geometry>
+      <material name="s5max_dark_grey"/>
+    </visual>
+  </link>
+  <joint name="dock_ir_right_joint" type="fixed">
+    <parent link="base_link"/>
+    <child link="dock_ir_right_link"/>
+    <origin xyz="${dock_ir_right_x} ${dock_ir_right_y} ${body_height / 2}" rpy="0 0 ${dock_ir_right_yaw}"/>
+  </joint>
+  <link name="dock_ir_right_link">
+    <visual>
+      <geometry>
+        <box size="0.006 0.020 0.012"/>
+      </geometry>
+      <material name="s5max_dark_grey"/>
+    </visual>
+  </link>
 </robot>
